File: ElectronicClock.sch (KiCad schematic (older format))
At the start: 53 parts

Commit message: Added some more components
Parts:
- removed DP? (x2): 7SEGMENTS, symbol 7SEGMENTS
- removed R? (x14): R, symbol R
- removed U? (x2): 74LS08, symbol 74LS08
- removed U? (x2): 74LS93, symbol 74LS93
- removed U? (x2): 74LS47, symbol 74LS47
- added D? (x2): D, symbol D
- added DP? (x4): 7SEGMENTS, symbol 7SEGMENTS
- added R? (x40): R, symbol R
- added SW? (x6): SW_Push, symbol SW_Push
- added SW? (x2): SW_DPDT_x2, symbol SW_DPDT_x2
- added unit 2 of U4
- added unit 3 of U4
- added U? (x4): 74LS93, symbol 74LS93
- added U? (x4): 74LS47, symbol 74LS47
- added U?: 74LS08, symbol 74LS08
- gave numbers to parts that had none: 1
Connections:
- net GND: now also U?.14 (CP0), U?.6 (D), R?.1, R?.1, R?.1, R?.1, R?.1, R?.1, SW?.1 (A), U4.7 (GND), U4.7 (GND), U?.14 (CP0), U?.14 (CP0), U?.2 (C), U?.6 (D), U?.6 (D), U?.7 (GND), U?.8 (GND), U?.8 (GND), U?.8 (GND), U?.8 (GND)
- net VCC: now also DP?.3 (C.A.), DP?.3 (C.A.), DP?.3 (C.A.), DP?.3 (C.A.), DP?.3 (C.A.), DP?.3 (C.A.), R?.1, R?.1, R?.1, R?.1, R?.1, R?.1, SW?.3 (C), SW?.6 (C), U4.14 (VCC), U4.14 (VCC), U?.14 (VCC), U?.16 (VCC), U?.16 (VCC), U?.16 (VCC), U?.16 (VCC), U?.5 (VCC), U?.5 (VCC), U?.5 (VCC), U?.5 (VCC)
- net 1/10Hz: now reaches U4.3, U?.1 (CP1..3)
- net at U?.4: now also U?.1 (B), U?.8 (Q2)
- net at U?.5: now also U?.2 (C), U?.8 (Q2)
- net HRST: now reaches U?.6
- net HRST: now also D?.2 (A), D?.2 (A), U?.2 (R0(1)), U?.3 (R0(2))
- net 1/60Hz: now reaches U4.11
- net 1/60Hz: now also U?.14 (CP0)
- net at U4.12: now also U?.1 (B), U?.2 (R0(1)), U?.8 (Q2)
- net at U4.13: now also U?.11 (Q3), U?.2 (C), U?.3 (R0(2))
- net at U?.7 (A), U?.9 (Q1): no longer U?.2 (R0(1))
- net at U?.3 (LT): now also U?.4 (BI), U?.5 (RBI), R?.2 (x2)
- net TSET: now reaches IC?.12 (RES), R?.1
- net TSET: now also SW?.2 (B)
- new net: U4.4, U?.1 (B), U?.2 (R0(1)), U?.9 (Q1)
- new net: U4.5, U?.11 (Q3), U?.3 (R0(2)), U?.6 (D)
- new net: U4.10, U?.11 (Q3), U?.2 (C), U?.3 (R0(2))
- new net: U4.9, U?.1 (B), U?.2 (R0(1)), U?.8 (Q2)
- new net: U?.1 (CP1..3), U?.12 (Q0), U?.7 (A) (x2)
- new net: U?.2 (C), U?.8 (Q2)
- new net: U?.7 (A), U?.9 (Q1) (x2)
- new net: R?.1, U?.10 (d) (x4)
- new net: R?.1, U?.11 (c) (x4)
- new net: R?.1, U?.12 (b) (x4)
- new net: R?.1, U?.13 (a) (x4)
- new net: R?.1, U?.14 (g) (x4)
- new net: R?.1, U?.15 (f) (x4)
- new net: R?.2, U?.3 (LT), U?.4 (BI), U?.5 (RBI) (x4)
- new net: R?.1, U?.9 (e) (x4)
- new net: DP?.1 (e), R?.2 (x4)
- new net: DP?.10 (g), R?.2 (x4)
- new net: DP?.2 (d), R?.2 (x4)
- new net: DP?.4 (c), R?.2 (x4)
- new net: DP?.6 (b), R?.2 (x4)
- new net: DP?.7 (a), R?.2 (x4)
- new net: DP?.9 (f), R?.2 (x4)
- new net: D?.1 (K), U?.1, U?.1 (B), U?.2 (R0(1)), U?.9 (Q1)
- new net: D?.1 (K), U?.11 (Q3), U?.2, U?.3 (R0(2)), U?.6 (D)
- new net: SW?.1, SW?.1, SW?.1, SW?.1, SW?.1, SW?.1, SW?.5 (B)
- new net: R?.2, SW?.2 (x6)
- new net 1/36000Hz: U?.1 (CP1..3), U?.3
- new net 1/3600Hz: U4.8, U?.14 (CP0)
- new net 1/600Hz: U4.6, U?.1 (CP1..3)
- no-connect marks 13 -> 28
Other:
- moved on the sheet: DP?, U4A, U4D, U?, U?B
