File: ElectronicClock.kicad_pcb (KiCad board)
At the start: 2 copper layers, 91 parts, among them IC1 4060N, SW1 SW_Push, SW2 SW_Push, SW3 SW_DPDT_x2, SW4 SW_Push, SW5 SW_Push, SW6 SW_Push, SW7 SW_Push, U1 74LS93, U10 74LS47, U11 74LS08, U12 74LS93, U13 74LS47, U14 74LS93, U15 74LS47, U2 74LS47, U3 74LS73, U4 74LS08, U5 74LS93, U6 74LS47, U7 74LS93, U8 74LS93, U9 74LS47, Y1 Crystal

Commit message: Reworked the component names
Parts:
- removed C2: 22p, Capacitors_THT:C_Disc_D3.0mm_W2.0mm_P2.50mm
- removed DP1, DP2, DP3, DP4, DP5, DP6: 7SEGMENTS, Displays_7-Segment:7SegmentLED_LTS6760_LTS6780
- removed IC1: 4060N, Housings_DIP:DIP-16_W7.62mm_Socket_LongPads
- removed R57: 1k, Resistors_THT:R_Axial_DIN0204_L3.6mm_D1.6mm_P7.62mm_Horizontal
- removed SW7: SW_Push, Buttons_Switches_THT:SW_PUSH_6mm
- removed U10, U13, U15, U6, U9: 74LS47, Housings_DIP:DIP-16_W7.62mm_Socket_LongPads
- removed U11, U4: 74LS08, Housings_DIP:DIP-14_W7.62mm_Socket_LongPads
- removed U12, U14, U5, U7, U8: 74LS93, Housings_DIP:DIP-14_W7.62mm_Socket_LongPads
- removed Y1: Crystal, Crystals:Crystal_DS10_d1.0mm_l4.3mm_Horizontal_1EP_style1
- added C0: 10p, Capacitors_THT:C_Disc_D3.0mm_W2.0mm_P2.50mm, F.Cu at (48.3, 142.2)
- added CTR_H0: 74LS93, Housings_DIP:DIP-14_W7.62mm_Socket_LongPads, F.Cu at (104.1, 76.2)
- added CTR_H1: 74LS93, Housings_DIP:DIP-14_W7.62mm_Socket_LongPads, F.Cu at (91.4, 76.2)
- added CTR_M0: 74LS93, Housings_DIP:DIP-14_W7.62mm_Socket_LongPads, F.Cu at (78.7, 76.2)
- added CTR_M1: 74LS93, Housings_DIP:DIP-14_W7.62mm_Socket_LongPads, F.Cu at (66.0, 76.2)
- added CTR_S0: 74LS93, Housings_DIP:DIP-14_W7.62mm_Socket_LongPads, F.Cu at (53.3, 76.2)
- added CTR_S1: 74LS93, Housings_DIP:DIP-14_W7.62mm_Socket_LongPads, F.Cu at (40.6, 76.2)
- added DP_H0: 7SEGMENTS, Displays_7-Segment:7SegmentLED_LTS6760_LTS6780, F.Cu at (48.3, 111.8)
- added DP_H1: 7SEGMENTS, Displays_7-Segment:7SegmentLED_LTS6760_LTS6780, F.Cu at (35.6, 111.8)
- added DP_M0: 7SEGMENTS, Displays_7-Segment:7SegmentLED_LTS6760_LTS6780, F.Cu at (83.8, 111.8)
- added DP_M1: 7SEGMENTS, Displays_7-Segment:7SegmentLED_LTS6760_LTS6780, F.Cu at (71.1, 111.8)
- added DP_S0: 7SEGMENTS, Displays_7-Segment:7SegmentLED_LTS6760_LTS6780, F.Cu at (119.4, 111.8)
- added DP_S1: 7SEGMENTS, Displays_7-Segment:7SegmentLED_LTS6760_LTS6780, F.Cu at (106.7, 111.8)
- added DRV_H0: 74LS47, Housings_DIP:DIP-16_W7.62mm_Socket_LongPads, F.Cu at (106.7, 50.8)
- added DRV_H1: 74LS47, Housings_DIP:DIP-16_W7.62mm_Socket_LongPads, F.Cu at (119.4, 50.8)
- added DRV_M0: 74LS47, Housings_DIP:DIP-16_W7.62mm_Socket_LongPads, F.Cu at (132.1, 50.8)
- added DRV_M1: 74LS47, Housings_DIP:DIP-16_W7.62mm_Socket_LongPads, F.Cu at (144.8, 50.8)
- added DRV_S0: 74LS47, Housings_DIP:DIP-16_W7.62mm_Socket_LongPads, F.Cu at (157.5, 50.8)
- added DRV_S1: 74LS47, Housings_DIP:DIP-16_W7.62mm_Socket_LongPads, F.Cu at (170.2, 50.8)
- added R0: 10M, Resistors_THT:R_Axial_DIN0204_L3.6mm_D1.6mm_P7.62mm_Horizontal, F.Cu at (106.7, 137.2)
- added SW0: SW_DPDT_x2, switch_dpdt:SWITCH_DPDT_8x8mm, F.Cu at (132.1, 83.8)
- added U0: 4060N, Housings_DIP:DIP-16_W7.62mm_Socket_LongPads, F.Cu at (190.5, 78.7)
- added X1: Crystal, Crystals:Crystal_DS10_d1.0mm_l4.3mm_Horizontal_1EP_style1, F.Cu at (63.5, 147.3)
- C1: value 10p -> 22p
- R12, R13, R14, R15, R18, R22: value 10k -> 1k
- R2: value 10M -> 10k
- R4, R5, R6, R7, R8: value 1k -> 10k
- SW3: value SW_DPDT_x2 -> SW_Push; footprint switch_dpdt:SWITCH_DPDT_8x8mm -> Buttons_Switches_THT:SW_PUSH_6mm
- U1: value 74LS93 -> 74LS73
- U2: value 74LS47 -> 74LS08; footprint Housings_DIP:DIP-16_W7.62mm_Socket_LongPads -> Housings_DIP:DIP-14_W7.62mm_Socket_LongPads
- U3: value 74LS73 -> 74LS08
- moved SW4 334.2 mm to (30.5, 167.6), turned to 0 degrees
- moved SW5 330.7 mm to (45.7, 170.2), turned to 0 degrees
- moved SW6 319.2 mm to (68.6, 170.2), turned to 0 degrees
- moved SW2 308.0 mm to (45.7, 160.0), turned to 0 degrees
- moved SW3 305.1 mm to (30.5, 157.5)
- moved R22 296.8 mm to (90.1, 138.0), turned to 0 degrees
- moved R18 287.2 mm to (90.1, 138.0), turned to 0 degrees
- moved SW1 278.4 mm to (68.6, 160.0), turned to 0 degrees
- moved R15 277.6 mm to (90.1, 138.0), turned to 0 degrees
- moved R14 268.1 mm to (90.1, 138.0), turned to 0 degrees
- moved R19 268.0 mm to (90.1, 138.0)
- moved R26 267.0 mm to (90.1, 138.0)
- moved R44 266.1 mm to (90.1, 138.0)
- moved R45 265.3 mm to (90.1, 138.0)
- moved R51 264.6 mm to (90.1, 138.0)
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Connections:
- D1 pad 1: Net-(D1-Pad1) -> Net-(CTR_H0-Pad11)
- D2 pad 1: Net-(D2-Pad1) -> Net-(CTR_H0-Pad2)
- R1 pad 1: Net-(IC1-Pad11) -> Net-(R0-Pad2)
- R1 pad 2: Net-(C1-Pad1) -> Net-(C0-Pad1)
- R10 pad 1: Net-(R10-Pad1) -> VCC
- R11 pad 1: Net-(R11-Pad1) -> VCC
- R12 pad 1: GND -> VCC
- R12 pad 2: 1Hz -> Net-(DRV_M1-Pad3)
- R13 pad 1: GND -> VCC
- R13 pad 2: 1/10Hz -> Net-(DRV_H0-Pad3)
- R14 pad 1: GND -> VCC
- R14 pad 2: 1/60Hz -> Net-(DRV_H1-Pad3)
- R15 pad 1: GND -> Net-(DRV_S0-Pad14)
- R15 pad 2: 1/600Hz -> Net-(DP_S0-Pad10)
- R16 pad 1: VCC -> Net-(DRV_S0-Pad15)
- R18 pad 1: GND -> Net-(DRV_S0-Pad10)
- R18 pad 2: 1/3600Hz -> Net-(DP_S0-Pad2)
- R2 pad 1: Net-(C2-Pad1) -> TSET
- R2 pad 2: Net-(IC1-Pad11) -> GND
- R22 pad 1: GND -> Net-(DRV_S1-Pad14)
- R22 pad 2: 1/36000Hz -> Net-(DP_S1-Pad10)
- R26 pad 1: VCC -> Net-(DRV_S1-Pad11)
- R3 pad 1: TSET -> GND
- R3 pad 2: GND -> 1Hz
- R31 pad 1: VCC -> Net-(DRV_M0-Pad9)
- R4 pad 1: VCC -> GND
- R4 pad 2: Net-(R4-Pad2) -> 1/10Hz
- R42 pad 1: VCC -> Net-(DRV_M1-Pad13)
- R43 pad 1: VCC -> Net-(DRV_H0-Pad14)
- R5 pad 1: Net-(R5-Pad1) -> GND
- R5 pad 2: Net-(DP1-Pad10) -> 1/60Hz
- R6 pad 1: Net-(R6-Pad1) -> GND
- R6 pad 2: Net-(DP1-Pad9) -> 1/600Hz
- R7 pad 1: Net-(R7-Pad1) -> GND
- R7 pad 2: Net-(DP1-Pad1) -> 1/3600Hz
- R8 pad 1: Net-(R8-Pad1) -> GND
- R8 pad 2: Net-(DP1-Pad2) -> 1/36000Hz
- R9 pad 1: Net-(R9-Pad1) -> VCC
- SW1 pad 1: Net-(SW1-Pad1) -> Net-(SW0-Pad5)
- SW2 pad 1: Net-(SW1-Pad1) -> Net-(SW0-Pad5)
- SW3 pad 1: GND -> Net-(SW0-Pad5)
- SW3 pad 2: TSET -> 1/60Hz
- SW4 pad 1: Net-(SW1-Pad1) -> Net-(SW0-Pad5)
- SW4 pad 2: 1/60Hz -> 1/600Hz
- SW5 pad 1: Net-(SW1-Pad1) -> Net-(SW0-Pad5)
- SW5 pad 2: 1/600Hz -> 1/3600Hz
- SW6 pad 1: Net-(SW1-Pad1) -> Net-(SW0-Pad5)
- SW6 pad 2: 1/3600Hz -> 1/36000Hz
- U1 pad 1: Net-(U1-Pad1) -> (no net)
- U1 pad 10: Net-(U1-Pad10) -> VCC
- U1 pad 11: Net-(U1-Pad11) -> GND
- U1 pad 12: Net-(U1-Pad1) -> (no net)
- U1 pad 14: 1Hz -> (no net)
- U1 pad 2: Net-(U1-Pad2) -> (no net)
- U1 pad 3: Net-(U1-Pad11) -> (no net)
- U1 pad 4: (no net) -> VCC
- U1 pad 5: VCC -> Net-(U0-Pad4)
- U1 pad 6: (no net) -> VCC
- U1 pad 7: (no net) -> VCC
- U1 pad 9: Net-(U1-Pad2) -> 1Hz
- U2 pad 1: Net-(U1-Pad2) -> Net-(CTR_S0-Pad2)
- U2 pad 10: Net-(R8-Pad1) -> Net-(CTR_M1-Pad11)
- U2 pad 11: Net-(R9-Pad1) -> 1/60Hz
- U2 pad 12: Net-(R10-Pad1) -> Net-(CTR_S1-Pad2)
- U2 pad 13: Net-(R11-Pad1) -> Net-(CTR_S1-Pad11)
- U2 pad 14: Net-(R5-Pad1) -> VCC
- U2 pad 2: Net-(U1-Pad8) -> Net-(CTR_S0-Pad11)
- U2 pad 3: Net-(R4-Pad2) -> 1/10Hz
- U2 pad 4: Net-(R4-Pad2) -> Net-(CTR_M0-Pad2)
- U2 pad 5: Net-(R4-Pad2) -> Net-(CTR_M0-Pad11)
- U2 pad 6: Net-(U1-Pad11) -> 1/600Hz
- U2 pad 7: Net-(U1-Pad1) -> GND
- U2 pad 8: GND -> 1/3600Hz
- U2 pad 9: Net-(R7-Pad1) -> Net-(CTR_M1-Pad2)
- U3 pad 1: (no net) -> Net-(CTR_H0-Pad2)
- U3 pad 10: VCC -> (no net)
- U3 pad 11: GND -> (no net)
- U3 pad 14: (no net) -> VCC
- U3 pad 2: (no net) -> Net-(CTR_H0-Pad11)
- U3 pad 3: (no net) -> 1/36000Hz
- U3 pad 4: VCC -> Net-(CTR_H1-Pad8)
- U3 pad 6: VCC -> HRST
- U3 pad 7: VCC -> GND
- U3 pad 8: Net-(U3-Pad8) -> (no net)
- U3 pad 9: 1Hz -> (no net)
Routing:
- net Net-(SW1-Pad1): track 77.4 -> 0.00 mm
- net Net-(C2-Pad1): track 24.4 -> 0.00 mm
- net VCC: track 17.3 -> 0.00 mm
- net Net-(IC1-Pad11): track 10.7 -> 0.00 mm
- net TSET: track 10.5 -> 0.00 mm
- net Net-(C1-Pad1): track 7.62 -> 0.00 mm
- net Net-(CTR_H0-Pad8): track 6.35 -> 0.00 mm
- net 1Hz: track 4.05 -> 0.00 mm
- net 1/60Hz: track 4.05 -> 0.00 mm
- net 1/600Hz: track 4.05 -> 0.00 mm
- net 1/3600Hz: track 4.05 -> 0.00 mm
- net 1/36000Hz: track 4.05 -> 0.00 mm
- net 1/10Hz: track 4.05 -> 0.00 mm

Commit message: Routed 3 displays
Parts:
- moved C0 246.1 mm to (271.8, 39.4)
- moved C1 244.1 mm to (271.8, 43.2)
- moved SW4 240.4 mm to (267.3, 126.4), turned to 90 degrees
- moved SW5 236.5 mm to (278.1, 126.4), turned to 90 degrees
- moved X1 231.8 mm to (269.2, 40.6), turned to 270 degrees
- moved SW3 228.2 mm to (256.5, 126.4), turned to 90 degrees
- moved SW6 224.7 mm to (288.9, 126.4), turned to 90 degrees
- moved R8 204.6 mm to (294.6, 139.7), turned to 90 degrees
- moved SW2 202.8 mm to (245.7, 126.4), turned to 90 degrees
- moved R7 194.4 mm to (284.5, 139.7), turned to 90 degrees
- moved R6 183.0 mm to (273.1, 139.7), turned to 90 degrees
- moved R2 180.1 mm to (252.7, 36.8)
- moved R1 177.2 mm to (252.7, 39.4)
- moved R0 174.4 mm to (252.7, 41.9)
- moved R5 172.8 mm to (262.9, 139.7), turned to 90 degrees
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Routing:
- net Net-(SW0-Pad5): track 0.00 -> 86.7 mm
- net Net-(DP_S0-Pad9): track 0.00 -> 38.7 mm
- net Net-(DP_S0-Pad10): track 0.00 -> 38.3 mm
- net Net-(DP_S1-Pad10): track 0.00 -> 32.6 mm
- net Net-(DP_M0-Pad9): track 0.00 -> 31.5 mm
- net Net-(DP_M0-Pad10): track 0.00 -> 31.0 mm
- net Net-(DP_S1-Pad9): track 0.00 -> 29.7 mm
- net Net-(DP_S0-Pad2): track 0.00 -> 29.1 mm
- net Net-(DP_S0-Pad1): track 0.00 -> 29.1 mm
- net Net-(DP_S0-Pad4): track 0.00 -> 28.0 mm
- net Net-(DP_S1-Pad4): track 0.00 -> 26.5 mm
- net Net-(DP_S1-Pad2): track 0.00 -> 26.5 mm
- net Net-(DP_S1-Pad1): track 0.00 -> 26.5 mm
- net Net-(C1-Pad1): track 0.00 -> 26.1 mm
- net Net-(DP_M0-Pad4): track 0.00 -> 25.9 mm
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Other:
- net class DISP added: clearance 0.2, trace_width 0.254, via_dia 0.6, via_drill 0.4
- net class Default: trace_width 0.5 -> 0.38
